File: kicad/RFID HW Detector - Rita/RFID HW Detector - Rita.kicad_pcb (KiCad board)
At the start: 2 copper layers, 17 parts, among them P1 CONN_01X04, SW1 SPST, SW2 SPST, SW3 SPST, SW4 SPST, SW5 SPST

Commit message: fixed circutboard
Parts:
- moved D5 3.25 mm to (213.4, 87.6), turned to 90 degrees
- moved D3 3.15 mm to (198.1, 87.6), turned to 90 degrees
- moved D2 3.15 mm to (191.1, 87.6), turned to 90 degrees
- moved D1 3.15 mm to (184.2, 87.6), turned to 90 degrees
- moved D4 3.14 mm to (205.7, 87.6), turned to 90 degrees
- renumbered D11 to D2
Connections:
- D2 pad 1: Net-(D2-Pad1) -> Net-(D1-Pad1)
- D2 pad 2: Net-(D1-Pad2) -> Net-(D2-Pad2)
- D3 pad 1: Net-(D3-Pad1) -> Net-(D1-Pad1)
- D3 pad 2: Net-(D1-Pad2) -> Net-(D3-Pad2)
- D4 pad 1: Net-(D4-Pad1) -> Net-(D1-Pad1)
- D4 pad 2: Net-(D1-Pad2) -> Net-(D4-Pad2)
- D5 pad 1: Net-(D5-Pad1) -> Net-(D1-Pad1)
- D5 pad 2: Net-(D1-Pad2) -> Net-(D5-Pad2)
- P1 pad 4: Net-(D1-Pad2) -> Net-(D1-Pad1)
- R1 pad 1: Net-(D1-Pad1) -> Net-(D1-Pad2)
- R2 pad 1: Net-(D2-Pad1) -> Net-(D2-Pad2)
- R3 pad 1: Net-(D3-Pad1) -> Net-(D3-Pad2)
- R4 pad 1: Net-(D4-Pad1) -> Net-(D4-Pad2)
- R5 pad 1: Net-(D5-Pad1) -> Net-(D5-Pad2)
- SHIELD1 pad GND2: Net-(D1-Pad2) -> Net-(D1-Pad1)
- SW1 pad 2: Net-(P1-Pad1) -> Net-(D1-Pad1)
- SW2 pad 2: Net-(P1-Pad1) -> Net-(D1-Pad1)
- SW3 pad 2: Net-(P1-Pad1) -> Net-(D1-Pad1)
- SW4 pad 2: Net-(P1-Pad1) -> Net-(D1-Pad1)
- SW5 pad 2: Net-(P1-Pad1) -> Net-(D1-Pad1)
Routing:
- net Net-(D1-Pad1): track 3.50 -> 284.4 mm
- net Net-(D1-Pad2): track 147.4 -> 4.23 mm
- net Net-(P1-Pad1): track 198.9 -> 130.3 mm
- net Net-(D5-Pad2): track 0.00 -> 5.42 mm
- net Net-(D4-Pad2): track 0.00 -> 4.44 mm
- net Net-(D3-Pad2): track 0.00 -> 4.25 mm
- net Net-(D5-Pad1): track 4.14 -> 0.00 mm
- net Net-(D2-Pad2): track 0.00 -> 4.14 mm
- net Net-(D4-Pad1): track 3.75 -> 0.00 mm
- net Net-(D2-Pad1): track 3.51 -> 0.00 mm
- net Net-(D3-Pad1): track 3.50 -> 0.00 mm
- net Net-(R5-Pad2): track 20.9 -> 18.0 mm
