File: kicad/RFID HW Detector - Rita/RFID HW Detector - Rita.sch (KiCad schematic (older format))
At the start: 17 parts, among them P1 CONN_01X04, SW1 SPST, SW2 SPST, SW3 SPST, SW4 SPST, SW5 SPST

Commit message: fixed circutboard
Connections:
- net at SW1.2, SW2.2, SW3.2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: now also P1.4 (P4), SHIELD1.GND2; no longer P1.1 (P1), SHIELD1.5V
- net at R4.1: now also D4.2 (A); no longer D4.1 (K)
- net at R5.1: now also D5.2 (A); no longer D5.1 (K)
- net at R3.1: now also D3.2 (A); no longer D3.1 (K)
- net at R2.1: now also D2.2 (A); no longer D2.1 (K)
- net at R1.1: now also D1.2 (A); no longer D1.1 (K)
- new net: P1.1 (P1), SHIELD1.5V
Changed lines of the file:
@@
 LIBS:contrib
 LIBS:valves
-LIBS:arduino_shieldsNCL
+LIBS:RFID HW Detector - Rita-cache
 EELAYER 25 0
 EELAYER END
@@
 F 3 "" H 8700 4500 50  0000 C CNN
 	1    8700 4500
-	1    0    0    -1
+	-1   0    0    1
 $EndComp
 $Comp
@@
 F 3 "" H 8700 4800 50  0000 C CNN
 	1    8700 4800
-	1    0    0    -1
+	-1   0    0    1
 $EndComp
 $Comp
@@
 F 3 "" H 8700 5100 50  0000 C CNN
 	1    8700 5100
-	1    0    0    -1
+	-1   0    0    1
 $EndComp
 $Comp
@@
 F 3 "" H 8700 5400 50  0000 C CNN
 	1    8700 5400
-	1    0    0    -1
+	-1   0    0    1
 $EndComp
 $Comp
@@
 F 3 "" H 8700 4200 50  0000 C CNN
 	1    8700 4200
-	1    0    0    -1
+	-1   0    0    1
 $EndComp
 $Comp
@@
 	6500 5400 7850 5400
 Wire Wire Line
-	8150 5400 8500 5400
-Wire Wire Line
-	8150 5100 8500 5100
-Wire Wire Line
-	8500 4800 8150 4800
-Wire Wire Line
-	8150 4500 8500 4500
-Wire Wire Line
-	8150 4200 8500 4200
-Wire Wire Line
 	7850 5100 6400 5100
 Wire Wire Line
@@
 	7700 4200 7850 4200
 Wire Wire Line
-	8900 4200 8900 6000
-Connection ~ 8900 4200
-Connection ~ 8900 4500
-Connection ~ 8900 4800
-Connection ~ 8900 5100
-Connection ~ 8900 5400
-Wire Wire Line
 	4450 4550 3650 4550
 Wire Wire Line
@@
 	7100 3950 6350 3950
 Wire Wire Line
-	8850 1100 8850 3650
+	8850 1750 8850 3650
 Connection ~ 8850 2800
 Connection ~ 8850 3250
 Connection ~ 8850 2400
 Connection ~ 8850 3650
-Wire Wire Line
-	8850 3650 9050 3650
-Wire Wire Line
-	9050 3650 9050 6200
-Wire Wire Line
-	9050 6200 3550 6200
-Wire Wire Line
-	3550 6200 3550 4350
-Wire Wire Line
-	3550 4350 4450 4350
 Connection ~ 8850 2050
 Wire Wire Line
-	8850 1100 7800 1100
-Wire Wire Line
-	7800 1100 7800 1300
-Wire Wire Line
-	8900 4200 9150 4200
-Wire Wire Line
-	9150 4200 9150 1000
-Wire Wire Line
-	9150 1000 6900 1000
-Wire Wire Line
-	6900 1000 6900 1600
-Wire Wire Line
-	6900 1600 7800 1600
+	7800 1300 6950 1300
+Wire Wire Line
+	6950 1300 6950 3450
+Wire Wire Line
+	6950 3450 4350 3450
+Wire Wire Line
+	4350 3450 4350 4350
+Wire Wire Line
+	4350 4350 4450 4350
+Wire Wire Line
+	8850 3650 8900 3650
+Wire Wire Line
+	7800 1600 7350 1600
+Wire Wire Line
+	7350 1600 7350 1750
+Wire Wire Line
+	7350 1750 8850 1750
+Wire Wire Line
+	8900 3650 8900 6000
+Wire Wire Line
+	8500 5400 8150 5400
+Wire Wire Line
+	8150 5100 8500 5100
+Wire Wire Line
+	8500 4800 8150 4800
+Wire Wire Line
+	8150 4500 8500 4500
+Wire Wire Line
+	8500 4200 8150 4200
 $EndSCHEMATC
